File: Blueprint1_hackpad.kicad_sch (KiCad schematic)
At the start: 0 parts

Commit message: TIME
pcb done
Parts:
- added Brd1: SSD1306, oled:SSD1306-0.91-OLED-4pin-128x32, symbol SSD1306-128x64_OLED:SSD1306
- added D1, D2, D3, D4, D5, D6, D7, D8: SK6812MINI, LED_SMD:LED_SK6812MINI_PLCC4_3.5x3.5mm_P1.75mm, symbol LED:SK6812MINI
- added SW1, SW2, SW3, SW4, SW5, SW6, SW7, SW8: SW_Push, Button_Switch_Keyboard:SW_Cherry_MX_1.00u_PCB, symbol Switch:SW_Push
- added U1: XIAO-RP2040-DIP, Seeed Studio XIAO Series Library:XIAO-RP2040-DIP, symbol Seeed_Studio_XIAO_Series:XIAO-RP2040-DIP
Connections:
- new net: SW2.1, U1.10 (GPIO4/MISO)
- new net: SW3.1, U1.9 (GPIO2/SCK)
- new net: SW4.1, U1.8 (GPIO1/RX)
- new net: D4.1 (DOUT), D5.3 (DIN)
- new net: D3.1 (DOUT), D4.3 (DIN)
- new net: D2.1 (DOUT), D3.3 (DIN)
- new net: SW5.2, U1.1 (GPIO26/ADC0/A0)
- new net: SW1.1, U1.11 (GPIO3/MOSI)
- new net: SW6.2, U1.2 (GPIO27/ADC1/A1)
- new net: SW7.2, U1.3 (GPIO28/ADC2/A2)
- new net: SW8.2, U1.4 (GPIO29/ADC3/A3)
- new net: Brd1.4 (SDA), U1.5 (GPIO6/SDA)
- new net: Brd1.3 (SCL), U1.6 (GPIO7/SCL)
- new net: D1.3 (DIN), U1.7 (GPIO0/TX)
- new net: D7.1 (DOUT), D8.3 (DIN)
- new net: D6.1 (DOUT), D7.3 (DIN)
- new net: D5.1 (DOUT), D6.3 (DIN)
- new net: D1.1 (DOUT), D2.3 (DIN)
- new net GND: Brd1.1 (GND), D1.2 (VSS), D2.2 (VSS), D3.2 (VSS), D4.2 (VSS), D5.2 (VSS), D6.2 (VSS), D7.2 (VSS), D8.2 (VSS), SW1.2, SW2.2, SW3.2, SW4.2, SW5.1, SW6.1, SW7.1, SW8.1, U1.13 (GND)
- new net vcc: Brd1.2 (VCC), D1.4 (VDD), D2.4 (VDD), D3.4 (VDD), D4.4 (VDD), D5.4 (VDD), D6.4 (VDD), D7.4 (VDD), D8.4 (VDD), U1.14 (VBUS)
